File: kicad/USB-pasthrough.kicad_sch (KiCad schematic)
At the start: 95 parts, among them J1 USB_Power, J10 MicroSD, J2 USB_C, J3 Power_Sel, J4 Cortex Debug, J5 SPI Display, J6 SWD, J7 Serial, J8 USB_A, J9 SD-1-A, SW1 Boot0, SW2 Reset, U1 AMS1117, U2 TPS2065C, U3 STM32F723VET6, Y1 8 MHz

Commit message: Add v0.2 gerbers and update PCB with silkscreen marks
Co-Authored-By: Claude Sonnet 4.6 <noreply@anthropic.com>
Parts:
- added C23: 10uF, Capacitor_SMD:C_0603_1608Metric_Pad1.08x0.95mm_HandSolder, symbol Device:C
- added C27: 100nF, Capacitor_SMD:C_0603_1608Metric_Pad1.08x0.95mm_HandSolder, symbol Device:C
- added TP10: VDDPHYHS, TestPoint:TestPoint_Pad_D1.0mm, symbol Connector:TestPoint
- renumbered C2 to C1, C14 to C12, C12 to C14, C19 to C15, C18 to C16, C15 to C17, C17 to C18, C16 to C19, C5 to C2, C24 to C20, C20 to C21, C21 to C22, C22 to C24, C23 to C25, C25 to C26, C6 to C3, C3 to C5, C1 to C6, ID2 to ID1, ID4 to ID2, ID5 to ID3, ID3 to ID4, ID1 to ID5, LED4 to LED3, LED3 to LED4, R2 to R1, R13 to R10, R9 to R11, R11 to R13, R1 to R2, R22 to R20, R20 to R22, R4 to R3, R3 to R4, R8 to R7, R10 to R8, R7 to R9, TP10 to TP13, TP13 to TP15, TP3 to TP2, TP2 to TP3, TP8 to TP7, TP7 to TP8
Connections:
- net +5V: now also C27.1
- net GND: now also C23.2, C27.2
- net VDDPHYHS: now reaches C21.1, C24.1, FB2.1, U3.54 (VDDPHYHS)
- net VDDPHYHS: now also TP10.1
- net VBUSA: now reaches J8.1 (VBUS), U2.1 (OUT)
- net VBUSA: now also C23.1
Other:
- moved on the sheet: J8, TP14, TP15, U2

Commit message: Sync bringup firmware and fix schematic for v0.2 bring-up
Bringup firmware (synced from ~/STM32F723_bringup):
- Remove PB15 GPIO test (was confusing USB host before PHY ready)
- Add GOTGCTL + DCTL to 2s status loop for ISR-safe debug
- VBDEN=1 empirically required for internal FS transceiver to drive D+
- BVALOEN+BVALOVAL=1 alongside VBDEN
- Fix PHY clock gate: only gate when low_power_enable=1
- OTG_HS IRQ priority 5, OTG_FS priority 6 (SWD/DAP preemption)
- rst=1 (ENUMDONE) confirmed on hub; v0.1 D+ trace physically broken

Schematic (post-fab corrections, not in v0.2-fab-send):
- Crystal label updated to 25 MHz (OTGPHYC PLLSEL=0x4)
- REXTPHYS corrected to 3K (was 12K; required for OTGPHYC impedance calibration)

Co-Authored-By: Claude Sonnet 4.6 <noreply@anthropic.com>
Parts:
- R15: value 12K -> 3K
- Y1: value 8 MHz -> 25 MHz
Changed lines of the file:
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@@
       (effects (font (size 1.27 1.27)) (justify right))
     )
-    (property "Value" "8 MHz" (id 1) (at 58.42 85.09 90)
+    (property "Value" "25 MHz" (id 1) (at 58.42 85.09 90)
       (effects (font (size 1.27 1.27)) (justify right))
     )
@@
     (in_bom yes) (on_board yes)
     (property "Reference" "R15" (id 0) (at 78.74 76.2 90))
-    (property "Value" "12K" (id 1) (at 78.74 81.28 90))
+    (property "Value" "3K" (id 1) (at 78.74 81.28 90))
     (property "Footprint" "Resistor_SMD:R_0603_1608Metric_Pad0.98x0.95mm_HandSolder" (id 2) (at 78.74 78.74 0)
       (effects (font (size 1.27 1.27)) hide)
@@
     )
     (path "/7e261482-6d94-42f1-947b-beece2e5a492"
-      (reference "R15") (unit 1) (value "12K") (footprint "Resistor_SMD:R_0603_1608Metric_Pad0.98x0.95mm_HandSolder")
+      (reference "R15") (unit 1) (value "3K") (footprint "Resistor_SMD:R_0603_1608Metric_Pad0.98x0.95mm_HandSolder")
     )
     (path "/21791df4-b3bc-4d1c-b633-6b787296d71d"
@@
     )
     (path "/5650e447-f5ae-4f8b-9d8d-8447b7a1abcd"
-      (reference "Y1") (unit 1) (value "8 MHz") (footprint "Crystal:Crystal_HC49-U_Vertical")
-    )
-  )
+      (reference "Y1") (unit 1) (value "25 MHz") (footprint "Crystal:Crystal_HC49-U_Vertical")
+    )
+  )

Commit message: Commit v0.2 KiCad schematic/PCB and library updates
- Schematic: xtal frequency updated to 25MHz, REXT to 3KΩ
- sym-lib-table: fix tps2065c to use relative ${KIPRJMOD} path
- fp-lib-table: add Library entry
- Add tps2065c.kicad_sym and SHF-105-01-F-D-TH connector library to kicad/libs/

Not tagged as sent-to-fab — schematic changes pending v0.2 board order.

Co-Authored-By: Claude Sonnet 4.6 <noreply@anthropic.com>
Parts:
- R15: value 3K -> 12K
- Y1: value 25 MHz -> 8 MHz
- renumbered ID5 to ID1, ID1 to ID2, ID4 to ID3, ID2 to ID4, ID3 to ID5
Connections:
- net RXD: now also U3.47 (PB11); no longer U3.25 (PA3)
- net TXD: now also U3.46 (PB10); no longer U3.24 (PA2)
Changed lines of the file:
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@@
   (no_connect (at 132.08 180.34))
   (no_connect (at 132.08 185.42))
-  (no_connect (at 132.08 129.54))
   (no_connect (at 132.08 109.22))
-  (no_connect (at 132.08 132.08))
   (no_connect (at 81.28 129.54))
   (no_connect (at 81.28 104.14))
+  (no_connect (at 132.08 68.58))
   (no_connect (at 132.08 160.02))
   (no_connect (at 81.28 96.52))
@@
   (no_connect (at 33.02 127))
   (no_connect (at 81.28 137.16))
+  (no_connect (at 132.08 66.04))
   (no_connect (at 81.28 93.98))
   (no_connect (at 81.28 127))
@@
     (effects (font (size 1.27 1.27)) (justify right bottom))
   )
-  (label "TXD" (at 132.08 66.04 0)
+  (label "TXD" (at 132.08 129.54 0)
     (effects (font (size 1.27 1.27)) (justify left bottom))
   )
@@
     (effects (font (size 1.27 1.27)) (justify left bottom))
   )
-  (label "RXD" (at 132.08 68.58 0)
+  (label "RXD" (at 132.08 132.08 0)
     (effects (font (size 1.27 1.27)) (justify left bottom))
   )
@@
   (symbol (lib_id "Jumper:Jumper_2_Bridged") (at 76.2 152.4 0) (mirror y) (unit 1)
     (in_bom yes) (on_board yes)
-    (property "Reference" "ID3" (id 0) (at 76.2 151.13 0))
+    (property "Reference" "ID5" (id 0) (at 76.2 151.13 0))
     (property "Value" "Jumper_2_Bridged" (id 1) (at 76.2 148.59 0)
       (effects (font (size 1.27 1.27)) hide)
@@
   (symbol (lib_id "Jumper:Jumper_2_Bridged") (at 76.2 147.32 0) (mirror y) (unit 1)
     (in_bom yes) (on_board yes)
-    (property "Reference" "ID4" (id 0) (at 76.2 146.05 0))
+    (property "Reference" "ID3" (id 0) (at 76.2 146.05 0))
     (property "Value" "Jumper_2_Bridged" (id 1) (at 76.2 143.51 0)
       (effects (font (size 1.27 1.27)) hide)
@@
       (effects (font (size 1.27 1.27)) (justify right))
     )
-    (property "Value" "25 MHz" (id 1) (at 58.42 85.09 90)
+    (property "Value" "8 MHz" (id 1) (at 58.42 85.09 90)
       (effects (font (size 1.27 1.27)) (justify right))
     )
@@
     (in_bom yes) (on_board yes)
     (property "Reference" "R15" (id 0) (at 78.74 76.2 90))
-    (property "Value" "3K" (id 1) (at 78.74 81.28 90))
+    (property "Value" "12K" (id 1) (at 78.74 81.28 90))
     (property "Footprint" "Resistor_SMD:R_0603_1608Metric_Pad0.98x0.95mm_HandSolder" (id 2) (at 78.74 78.74 0)
       (effects (font (size 1.27 1.27)) hide)
@@
   (symbol (lib_id "Jumper:Jumper_2_Bridged") (at 76.2 142.24 0) (mirror y) (unit 1)
     (in_bom yes) (on_board yes)
-    (property "Reference" "ID5" (id 0) (at 76.2 140.97 0))
+    (property "Reference" "ID1" (id 0) (at 76.2 140.97 0))
     (property "Value" "Jumper_2_Bridged" (id 1) (at 76.2 138.43 0)
       (effects (font (size 1.27 1.27)) hide)
@@
   (symbol (lib_id "Jumper:Jumper_2_Open") (at 76.2 144.78 0) (mirror y) (unit 1)
     (in_bom yes) (on_board yes)
-    (property "Reference" "ID1" (id 0) (at 76.2 143.51 0))
+    (property "Reference" "ID2" (id 0) (at 76.2 143.51 0))
     (property "Value" "Jumper_2_Bridged" (id 1) (at 76.2 140.97 0)
       (effects (font (size 1.27 1.27)) hide)
@@
   (symbol (lib_id "Jumper:Jumper_2_Bridged") (at 76.2 149.86 0) (mirror y) (unit 1)
     (in_bom yes) (on_board yes)
-    (property "Reference" "ID2" (id 0) (at 76.2 148.59 0))
+    (property "Reference" "ID4" (id 0) (at 76.2 148.59 0))
     (property "Value" "Jumper_2_Bridged" (id 1) (at 76.2 146.05 0)
       (effects (font (size 1.27 1.27)) hide)
@@
       (reference "H4") (unit 1) (value "MountingHole") (footprint "MountingHole:MountingHole_2.2mm_M2_Pad")
     )
-    (path "/a626e9e8-3375-4718-9ad8-d8caf9b074bb"
-      (reference "ID1") (unit 1) (value "Jumper_2_Bridged") (footprint "Jumper:SolderJumper-2_P1.3mm_Open_Pad1.0x1.5mm")
+    (path "/96e7b321-1a35-4bce-b54a-aba345801942"
+      (reference "ID1") (unit 1) (value "Jumper_2_Bridged") (footprint "Jumper:SolderJumper-2_P1.3mm_Bridged_Pad1.0x1.5mm")
     )
-    (path "/df8f3236-ca66-46c0-9b8f-22b38c82257e"
-      (reference "ID2") (unit 1) (value "Jumper_2_Bridged") (footprint "Jumper:SolderJumper-2_P1.3mm_Bridged_Pad1.0x1.5mm")
+    (path "/a626e9e8-3375-4718-9ad8-d8caf9b074bb"
+      (reference "ID2") (unit 1) (value "Jumper_2_Bridged") (footprint "Jumper:SolderJumper-2_P1.3mm_Open_Pad1.0x1.5mm")
     )
-    (path "/0adffc54-70e2-42c5-8aa7-e136dde5bc9e"
+    (path "/54720c1e-b373-4e5e-80dc-b8d36d988cb6"
       (reference "ID3") (unit 1) (value "Jumper_2_Bridged") (footprint "Jumper:SolderJumper-2_P1.3mm_Bridged_Pad1.0x1.5mm")
     )
-    (path "/54720c1e-b373-4e5e-80dc-b8d36d988cb6"
+    (path "/df8f3236-ca66-46c0-9b8f-22b38c82257e"
       (reference "ID4") (unit 1) (value "Jumper_2_Bridged") (footprint "Jumper:SolderJumper-2_P1.3mm_Bridged_Pad1.0x1.5mm")
     )
-    (path "/96e7b321-1a35-4bce-b54a-aba345801942"
+    (path "/0adffc54-70e2-42c5-8aa7-e136dde5bc9e"
       (reference "ID5") (unit 1) (value "Jumper_2_Bridged") (footprint "Jumper:SolderJumper-2_P1.3mm_Bridged_Pad1.0x1.5mm")
     )
@@
     )
     (path "/7e261482-6d94-42f1-947b-beece2e5a492"
-      (reference "R15") (unit 1) (value "3K") (footprint "Resistor_SMD:R_0603_1608Metric_Pad0.98x0.95mm_HandSolder")
+      (reference "R15") (unit 1) (value "12K") (footprint "Resistor_SMD:R_0603_1608Metric_Pad0.98x0.95mm_HandSolder")
     )
     (path "/21791df4-b3bc-4d1c-b633-6b787296d71d"
@@
     )
     (path "/5650e447-f5ae-4f8b-9d8d-8447b7a1abcd"
-      (reference "Y1") (unit 1) (value "25 MHz") (footprint "Crystal:Crystal_HC49-U_Vertical")
+      (reference "Y1") (unit 1) (value "8 MHz") (footprint "Crystal:Crystal_HC49-U_Vertical")
     )
   )
