File: kicad/USB-pasthrough.kicad_sch (KiCad schematic)
At the start: 98 parts, among them J1 USB_Power, J10 MicroSD, J2 USB_C, J3 Power_Sel, J4 Cortex Debug, J5 SPI Display, J6 SWD, J7 Serial, J8 USB_A, J9 SD-1-A, SW1 Boot0, SW2 Reset, U1 AMS1117, U2 TPS2065C, U3 STM32F723VET6, Y1 8 MHz

Commit message: Update cortex Debug connector footprint
Parts:
- J4: footprint Connector_PinHeader_1.27mm:PinHeader_2x05_P1.27mm_Vertical -> SHF-105-01-F-D-TH:SAMTEC_SHF-105-01-F-D-TH
Changed lines of the file:
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@@
     (property "Reference" "J4" (id 0) (at 172.72 109.22 0))
     (property "Value" "Cortex Debug" (id 1) (at 172.72 111.76 0))
-    (property "Footprint" "Connector_PinHeader_1.27mm:PinHeader_2x05_P1.27mm_Vertical" (id 2) (at 173.99 120.65 0)
+    (property "Footprint" "SHF-105-01-F-D-TH:SAMTEC_SHF-105-01-F-D-TH" (id 2) (at 173.99 120.65 0)
       (effects (font (size 1.27 1.27)) hide)
     )
@@
     )
     (path "/48e4579d-5e85-401f-9ce6-27ca1a2535a0"
-      (reference "J4") (unit 1) (value "Cortex Debug") (footprint "Connector_PinHeader_1.27mm:PinHeader_2x05_P1.27mm_Vertical")
+      (reference "J4") (unit 1) (value "Cortex Debug") (footprint "SHF-105-01-F-D-TH:SAMTEC_SHF-105-01-F-D-TH")
     )
     (path "/4908c02f-304f-4379-bc6d-3d980e650980"
