File: kicad/USB-pasthrough.kicad_sch (KiCad schematic)
At the start: 98 parts, among them J1 USB_Power, J10 MicroSD, J2 USB_C, J3 Power_Sel, J4 Cortex Debug, J5 SPI Display, J6 SWD, J7 Serial, J8 USB_A, J9 SD-1-A, SW1 Boot0, SW2 Reset, U1 AMS1117, U2 TPS2065C, U3 STM32F723VET6, Y1 8 MHz

Commit message: Update v0.2 LED current limit resistors for balanced brightness
Blue: 33Ω (~9mA, Vf~3.0V) — reference, matches v0.1
Yellow: 100Ω (~12mA, Vf~2.1V) — brighter than v0.1 150Ω
Green: 390Ω (~3mA, Vf~2.1V) — reduced for eye sensitivity compensation

All three on TIM1 CH1/2/3 PWM for firmware trim.

Co-Authored-By: Claude Sonnet 4.6 <noreply@anthropic.com>
Parts:
- R20: value 68 -> 390
- R22: value 150 -> 100
Changed lines of the file:
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@@
     (in_bom yes) (on_board yes) (fields_autoplaced)
     (property "Reference" "R20" (id 0) (at 248.92 81.28 90))
-    (property "Value" "68" (id 1) (at 248.92 83.82 90))
+    (property "Value" "390" (id 1) (at 248.92 83.82 90))
     (property "Footprint" "Resistor_SMD:R_0603_1608Metric_Pad0.98x0.95mm_HandSolder" (id 2) (at 248.92 87.63 0)
       (effects (font (size 1.27 1.27)) hide)
@@
     (in_bom yes) (on_board yes) (fields_autoplaced)
     (property "Reference" "R22" (id 0) (at 248.92 97.79 90))
-    (property "Value" "150" (id 1) (at 248.92 100.33 90))
+    (property "Value" "100" (id 1) (at 248.92 100.33 90))
     (property "Footprint" "Resistor_SMD:R_0603_1608Metric_Pad0.98x0.95mm_HandSolder" (id 2) (at 248.92 104.14 0)
       (effects (font (size 1.27 1.27)) hide)
@@
     )
     (path "/1a82aba1-7bcd-415b-b242-a8697f42897d"
-      (reference "R20") (unit 1) (value "68") (footprint "Resistor_SMD:R_0603_1608Metric_Pad0.98x0.95mm_HandSolder")
+      (reference "R20") (unit 1) (value "390") (footprint "Resistor_SMD:R_0603_1608Metric_Pad0.98x0.95mm_HandSolder")
     )
     (path "/d4e6855f-877c-4251-bf9e-698081c7e725"
@@
     )
     (path "/6e07490e-b1ba-4686-bc5c-17b021c96957"
-      (reference "R22") (unit 1) (value "150") (footprint "Resistor_SMD:R_0603_1608Metric_Pad0.98x0.95mm_HandSolder")
+      (reference "R22") (unit 1) (value "100") (footprint "Resistor_SMD:R_0603_1608Metric_Pad0.98x0.95mm_HandSolder")
     )
     (path "/7fb86b33-f6c8-4735-8ebb-bbd50db9e462"
