File: kicad/USB-pasthrough.kicad_sch (KiCad schematic)
At the start: 98 parts, among them J1 USB_Power, J10 MicroSD, J2 USB_C, J3 Power_Sel, J4 Cortex Debug, J5 SPI Display, J6 SWD, J7 Serial, J8 USB_A, J9 SD-1-A, SW1 Boot0, SW2 Reset, U1 AMS1117, U2 TPS2065C, U3 STM32F723VET6, Y1 8 MHz

Commit message: Make ground testpoints also alignment features
Parts:
- added TP16: GND, Alignment:TestPoint_THTPad_D2.0mm_Drill0.8mm_Align, symbol Connector:TestPoint
- TP1: footprint TestPoint:TestPoint_THTPad_D2.0mm_Drill1.0mm -> Alignment:TestPoint_THTPad_D2.0mm_Drill0.8mm_Align; Notes (none) -> Align feature
Connections:
- net GND: now also TP16.1
Changed lines of the file:
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@@
+    (pin "1")
+  )
+  (symbol (lib_id "power:GND") (at 43.18 90.17 0) (unit 1)
+    (in_bom yes) (on_board yes) (fields_autoplaced)
+    (property "Reference" "#PWR056" (id 0) (at 43.18 96.52 0)
+      (effects (font (size 1.27 1.27)) hide)
+    )
+    (property "Value" "GND" (id 1) (at 43.18 95.25 0))
+    (property "Footprint" "" (id 2) (at 43.18 90.17 0)
+      (effects (font (size 1.27 1.27)) hide)
+    )
+    (property "Datasheet" "" (id 3) (at 43.18 90.17 0)
+      (effects (font (size 1.27 1.27)) hide)
+    )
     (pin "1")
   )
@@
     (pin "1")
   )
+  (symbol (lib_name "TestPoint_2") (lib_id "Connector:TestPoint") (at 43.18 90.17 0) (unit 1)
+    (in_bom yes) (on_board yes)
+    (property "Reference" "TP16" (id 0) (at 45.72 85.5979 0)
+      (effects (font (size 1.27 1.27)) (justify left))
+    )
+    (property "Value" "GND" (id 1) (at 45.72 88.1379 0)
+      (effects (font (size 1.27 1.27)) (justify left))
+    )
+    (property "Footprint" "Alignment:TestPoint_THTPad_D2.0mm_Drill0.8mm_Align" (id 2) (at 48.26 90.17 0)
+      (effects (font (size 1.27 1.27)) hide)
+    )
+    (property "Datasheet" "~" (id 3) (at 48.26 90.17 0)
+      (effects (font (size 1.27 1.27)) hide)
+    )
+    (property "Notes" "Align feature" (id 4) (at 49.53 90.17 0))
+    (pin "1")
+  )
   (symbol (lib_name "MountingHole_3") (lib_id "Mechanical:MountingHole") (at 20.32 80.01 0) (unit 1)
     (in_bom yes) (on_board yes) (fields_autoplaced)
@@
   )
   (symbol (lib_name "TestPoint_2") (lib_id "Connector:TestPoint") (at 43.18 76.2 0) (unit 1)
-    (in_bom yes) (on_board yes) (fields_autoplaced)
+    (in_bom yes) (on_board yes)
     (property "Reference" "TP1" (id 0) (at 45.72 71.6279 0)
       (effects (font (size 1.27 1.27)) (justify left))
@@
       (effects (font (size 1.27 1.27)) (justify left))
     )
-    (property "Footprint" "TestPoint:TestPoint_THTPad_D2.0mm_Drill1.0mm" (id 2) (at 48.26 76.2 0)
+    (property "Footprint" "Alignment:TestPoint_THTPad_D2.0mm_Drill0.8mm_Align" (id 2) (at 48.26 76.2 0)
       (effects (font (size 1.27 1.27)) hide)
     )
@@
       (effects (font (size 1.27 1.27)) hide)
     )
+    (property "Notes" "Align feature" (id 4) (at 49.53 76.2 0))
     (pin "1")
   )
@@
       (reference "#PWR055") (unit 1) (value "GND") (footprint "")
     )
+    (path "/77db43a4-cfdb-4b4f-b9a9-ae493460b523"
+      (reference "#PWR056") (unit 1) (value "GND") (footprint "")
+    )
     (path "/2641c309-b1f2-413e-9bab-c17808f1d2ee"
       (reference "#PWR0101") (unit 1) (value "GND") (footprint "Resistor_SMD:R_0603_1608Metric_Pad0.98x0.95mm_HandSolder")
@@
     )
     (path "/c65cc65e-11e7-41cb-818c-ff91bd78cb55"
-      (reference "TP1") (unit 1) (value "GND") (footprint "TestPoint:TestPoint_THTPad_D2.0mm_Drill1.0mm")
+      (reference "TP1") (unit 1) (value "GND") (footprint "Alignment:TestPoint_THTPad_D2.0mm_Drill0.8mm_Align")
     )
     (path "/74d256c6-8769-4186-a255-1aea04864309"
@@
       (reference "TP15") (unit 1) (value "USBA+") (footprint "TestPoint:TestPoint_Pad_D1.0mm")
     )
+    (path "/ac3bf2fd-0ea3-41d3-9d1c-a58bf2caca08"
+      (reference "TP16") (unit 1) (value "GND") (footprint "Alignment:TestPoint_THTPad_D2.0mm_Drill0.8mm_Align")
+    )
     (path "/bb17c35c-a70d-4760-bafe-90e840af4fd7"
