File: kicad/USB-pasthrough.kicad_pcb (KiCad board)
At the start: 4 copper layers, 40 x 80 mm, 95 parts, among them J1 USB_Power, J10 MicroSD, J2 USB_C, J3 Power_Sel, J4 Cortex Debug, J5 SPI Display, J6 SWD, J7 Serial, J8 USB_A, J9 SD-1-A, SW1 Boot0, SW2 Reset, U1 AMS1117, U2 TPS2065C, U3 STM32F723VET6, Y1 8 MHz

Commit message: Schematic/PCB: connect PB13 to VBUS_DATA for OTG_HS VBUS sense
Completes v0.2 change list item 2 — enables OTG_HS VBUS comparator
so USB-C device D+ pull-up activates when VBUS is present.

Co-Authored-By: Claude Sonnet 4.6 <noreply@anthropic.com>
Connections:
- F2 pad 1: /VBUS_DATA -> /USBC_VBUS_DATA
- U3 pad 52: unconnected-(U3-Pad52) -> /USBC_VBUS_DATA
Routing:
- net /VBUS_DATA: track 3.94 -> 0.00 mm
- net /USBC_VBUS_DATA: track 0.00 -> 3.94 mm
Changed lines of the file:
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@@
   (net 74 "Net-(R18-Pad2)")
   (net 75 "Net-(R19-Pad1)")
-  (net 76 "Net-(U3-Pad67)")
+  (net 76 "/USBC_VBUS_DATA")
   (net 77 "unconnected-(U3-Pad98)")
   (net 78 "unconnected-(U3-Pad97)")
@@
   (net 90 "unconnected-(U3-Pad59)")
   (net 91 "unconnected-(U3-Pad58)")
-  (net 92 "unconnected-(U3-Pad52)")
+  (net 92 "Net-(TP7-Pad1)")
   (net 93 "unconnected-(U3-Pad51)")
   (net 94 "unconnected-(U3-Pad47)")
@@
     (fp_circle (center 0 0) (end 1 0) (layer "F.CrtYd") (width 0.05) (fill none))
     (pad "1" smd circle (at 0 0) (size 1 1) (layers "F.Cu" "F.Mask")
-      (net 76 "Net-(U3-Pad67)") (pinfunction "1") (pintype "passive"))
+      (net 92 "Net-(TP7-Pad1)") (pinfunction "1") (pintype "passive"))
   )
   (footprint "Connector_PinHeader_2.54mm:PinHeader_1x10_P2.54mm_Vertical" (layer "F.Cu")
@@
       (net 93 "unconnected-(U3-Pad51)") (pinfunction "PB12") (pintype "bidirectional+no_connect"))
     (pad "52" smd roundrect (at 7.675 5.5) (size 1.6 0.3) (layers "F.Cu" "F.Paste" "F.Mask") (roundrect_rratio 0.25)
-      (net 92 "unconnected-(U3-Pad52)") (pinfunction "PB13") (pintype "bidirectional+no_connect"))
+      (net 76 "/USBC_VBUS_DATA") (pinfunction "PB13") (pintype "bidirectional"))
     (pad "53" smd roundrect (at 7.675 5) (size 1.6 0.3) (layers "F.Cu" "F.Paste" "F.Mask") (roundrect_rratio 0.25)
       (net 72 "Net-(R15-Pad1)") (pinfunction "REXTPHYHS") (pintype "bidirectional"))
@@
       (net 49 "/SD1_D1") (pinfunction "PC9") (pintype "bidirectional"))
     (pad "67" smd roundrect (at 7.675 -2) (size 1.6 0.3) (layers "F.Cu" "F.Paste" "F.Mask") (roundrect_rratio 0.25)
-      (net 76 "Net-(U3-Pad67)") (pinfunction "PA8") (pintype "bidirectional"))
+      (net 92 "Net-(TP7-Pad1)") (pinfunction "PA8") (pintype "bidirectional"))
     (pad "68" smd roundrect (at 7.675 -2.5) (size 1.6 0.3) (layers "F.Cu" "F.Paste" "F.Mask") (roundrect_rratio 0.25)
       (net 84 "unconnected-(U3-Pad68)") (pinfunction "PA9") (pintype "bidirectional+no_connect"))
@@
     (fp_line (start -2.25 -1.6) (end 2.25 -1.6) (layer "F.Fab") (width 0.1))
     (pad "1" smd roundrect (at -2.225 0 180) (size 1.3 3.4) (layers "F.Cu" "F.Paste" "F.Mask") (roundrect_rratio 0.192308)
-      (net 11 "/VBUS_DATA") (pintype "passive"))
+      (net 76 "/USBC_VBUS_DATA") (pintype "passive"))
     (pad "2" smd roundrect (at 2.225 0 180) (size 1.3 3.4) (layers "F.Cu" "F.Paste" "F.Mask") (roundrect_rratio 0.192308)
       (net 12 "Net-(F2-Pad2)") (pintype "passive"))
@@
   (segment (start 104.6 62.575) (end 104.6 64.075) (width 1) (layer "F.Cu") (net 10))
   (segment (start 106.432 61.78) (end 105.395 61.78) (width 1) (layer "F.Cu") (net 10))
-  (segment (start 120.025 60.25) (end 119.805 60.47) (width 0.25) (layer "F.Cu") (net 11))
-  (segment (start 119.805 60.47) (end 119.805 64.1) (width 1) (layer "F.Cu") (net 11))
   (segment locked (start 116.9 57.75) (end 116.4 57.75) (width 0.5) (layer "F.Cu") (net 12))
   (segment locked (start 117.975 54.775) (end 117.975 56.125) (width 0.5) (layer "F.Cu") (net 12))
@@
   (segment (start 109.76 121.8) (end 109.76 120.623) (width 0.25) (layer "F.Cu") (net 75))
   (segment (start 109.76 120.623) (end 109.95 120.433) (width 0.25) (layer "F.Cu") (net 75))
-  (segment (start 133.75 86.725) (end 133.375 86.35) (width 0.25) (layer "F.Cu") (net 76))
-  (segment (start 127.675 88) (end 129.075216 88) (width 0.25) (layer "F.Cu") (net 76))
-  (segment (start 133.15 88.4) (end 133.75 87.8) (width 0.25) (layer "F.Cu") (net 76))
-  (segment (start 129.075216 88) (end 129.475216 88.4) (width 0.25) (layer "F.Cu") (net 76))
-  (segment (start 129.475216 88.4) (end 133.15 88.4) (width 0.25) (layer "F.Cu") (net 76))
-  (segment (start 133.75 87.8) (end 133.75 86.725) (width 0.25) (layer "F.Cu") (net 76))
+  (segment (start 120.025 60.25) (end 119.805 60.47) (width 0.25) (layer "F.Cu") (net 76))
+  (segment (start 119.805 60.47) (end 119.805 64.1) (width 1) (layer "F.Cu") (net 76))
+  (segment (start 133.75 86.725) (end 133.375 86.35) (width 0.25) (layer "F.Cu") (net 92))
+  (segment (start 127.675 88) (end 129.075216 88) (width 0.25) (layer "F.Cu") (net 92))
+  (segment (start 133.15 88.4) (end 133.75 87.8) (width 0.25) (layer "F.Cu") (net 92))
+  (segment (start 129.075216 88) (end 129.475216 88.4) (width 0.25) (layer "F.Cu") (net 92))
+  (segment (start 129.475216 88.4) (end 133.15 88.4) (width 0.25) (layer "F.Cu") (net 92))
+  (segment (start 133.75 87.8) (end 133.75 86.725) (width 0.25) (layer "F.Cu") (net 92))
   (zone (net 0) (net_name "") (layers "In1.Cu" "In2.Cu") (hatch edge 0.508)
     (connect_pads (clearance 0))

Commit message: Schematic/PCB: update signal names and complete PB13 VBUS_DATA routing
Co-Authored-By: Claude Sonnet 4.6 <noreply@anthropic.com>
Connections:
- F2 pad 1: /USBC_VBUS_DATA -> /VBUS_DATA
- U3 pad 52: /USBC_VBUS_DATA -> /VBUS_DATA
Routing:
- net /VBUS_DATA: track 0.00 -> 41.9 mm, vias 0 -> 2
- net /USBC_VBUS_DATA: track 3.94 -> 0.00 mm
- net /SD1_CDET: track 60.3 -> 57.1 mm
- net Net-(ID4-Pad1): track 17.8 -> 18.6 mm

Commit message: Add v0.2 gerbers and update PCB with silkscreen marks
Co-Authored-By: Claude Sonnet 4.6 <noreply@anthropic.com>
Parts:
- added C23: 10uF, Capacitor_SMD:C_0603_1608Metric_Pad1.08x0.95mm_HandSolder, F.Cu at (117.0, 113.7)
- added C27: 100nF, Capacitor_SMD:C_0603_1608Metric_Pad1.08x0.95mm_HandSolder, F.Cu at (112.8, 115.1)
- added TP10: VDDPHYHS, TestPoint:TestPoint_Pad_D1.0mm, F.Cu at (133.9, 95.5)
- moved TP7 12.1 mm to (115.9, 77.0)
- renumbered C2 to C1, C14 to C12, C12 to C14, C19 to C15, C18 to C16, C15 to C17, C17 to C18, C16 to C19, C5 to C2, C24 to C20, C20 to C21, C21 to C22, C22 to C24, C23 to C25, C25 to C26, C6 to C3, C3 to C5, C1 to C6, ID2 to ID1, ID4 to ID2, ID5 to ID3, ID3 to ID4, ID1 to ID5, LED4 to LED3, LED3 to LED4, R2 to R1, R13 to R10, R9 to R11, R11 to R13, R1 to R2, R22 to R20, R20 to R22, R4 to R3, R3 to R4, R8 to R7, R10 to R8, R7 to R9, TP10 to TP13, TP13 to TP15, TP3 to TP2, TP2 to TP3, TP8 to TP7, TP7 to TP8
Connections:
- net Net-(C20-Pad1) renamed /VDDPHYHS
- net Net-(J8-Pad1) renamed /VBUSA
Routing:
- net /SD1_D1: track 46.7 -> 27.5 mm
- net /SD1_CDET: track 57.1 -> 49.8 mm
- net /VDDPHYHS: track 8.48 -> 13.2 mm
- net GND: track 97.4 -> 100.2 mm, vias 52 -> 55
- net /VBUSA: track 8.31 -> 10.7 mm
- net +5V: track 79.7 -> 81.5 mm
- net /LED5_B: track 38.7 -> 40.1 mm
- net /LED5_R: track 45.2 -> 46.4 mm
- net /LCD_BL: track 40.0 -> 39.0 mm
- net /TXD: track 27.2 -> 26.5 mm
- net /RXD: track 27.2 -> 26.7 mm

Commit message: Sync bringup firmware and fix schematic for v0.2 bring-up
Bringup firmware (synced from ~/STM32F723_bringup):
- Remove PB15 GPIO test (was confusing USB host before PHY ready)
- Add GOTGCTL + DCTL to 2s status loop for ISR-safe debug
- VBDEN=1 empirically required for internal FS transceiver to drive D+
- BVALOEN+BVALOVAL=1 alongside VBDEN
- Fix PHY clock gate: only gate when low_power_enable=1
- OTG_HS IRQ priority 5, OTG_FS priority 6 (SWD/DAP preemption)
- rst=1 (ENUMDONE) confirmed on hub; v0.1 D+ trace physically broken

Schematic (post-fab corrections, not in v0.2-fab-send):
- Crystal label updated to 25 MHz (OTGPHYC PLLSEL=0x4)
- REXTPHYS corrected to 3K (was 12K; required for OTGPHYC impedance calibration)

Co-Authored-By: Claude Sonnet 4.6 <noreply@anthropic.com>
Parts:
- added REF**: OSHW-Logo2_7.3x6mm_Copper, Symbol:OSHW-Logo2_7.3x6mm_Copper, F.Cu at (130.0, 112.3)
- added REF**: KiCad-Logo2_5mm_SilkScreen, Symbol:KiCad-Logo2_5mm_SilkScreen, B.Cu at (126.3, 112.0)
Other:
- board text added: "USB-pasthrough V0.2 beattie@beattie-home.net"

Commit message: Commit v0.2 KiCad schematic/PCB and library updates
- Schematic: xtal frequency updated to 25MHz, REXT to 3KΩ
- sym-lib-table: fix tps2065c to use relative ${KIPRJMOD} path
- fp-lib-table: add Library entry
- Add tps2065c.kicad_sym and SHF-105-01-F-D-TH connector library to kicad/libs/

Not tagged as sent-to-fab — schematic changes pending v0.2 board order.

Co-Authored-By: Claude Sonnet 4.6 <noreply@anthropic.com>
Parts:
- renumbered ID5 to ID1, ID1 to ID2, ID4 to ID3, ID2 to ID4, ID3 to ID5
Changed lines of the file:
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@@
     (property "Sheetname" "")
     (attr exclude_from_pos_files)
-    (fp_text reference "ID1" (at 2.8 0 90) (layer "B.SilkS")
+    (fp_text reference "ID2" (at 2.8 0 90) (layer "B.SilkS")
       (effects (font (size 1 1) (thickness 0.15)) (justify mirror))
     )
@@
     (property "Sheetname" "")
     (attr exclude_from_pos_files)
-    (fp_text reference "ID2" (at 2.8 0.05 90) (layer "B.SilkS")
+    (fp_text reference "ID4" (at 2.8 0.05 90) (layer "B.SilkS")
       (effects (font (size 1 1) (thickness 0.15)) (justify mirror))
     )
@@
     (property "Sheetname" "")
     (attr exclude_from_pos_files)
-    (fp_text reference "ID3" (at 2.9 0.1 90) (layer "B.SilkS")
+    (fp_text reference "ID5" (at 2.9 0.1 90) (layer "B.SilkS")
       (effects (font (size 1 1) (thickness 0.15)) (justify mirror))
     )
@@
     (property "Sheetname" "")
     (attr exclude_from_pos_files)
-    (fp_text reference "ID4" (at 2.85 0.1 90) (layer "B.SilkS")
+    (fp_text reference "ID3" (at 2.85 0.1 90) (layer "B.SilkS")
       (effects (font (size 1 1) (thickness 0.15)) (justify mirror))
     )
@@
     (property "Sheetname" "")
     (attr exclude_from_pos_files)
-    (fp_text reference "ID5" (at 2.7 0.1 90) (layer "B.SilkS")
+    (fp_text reference "ID1" (at 2.7 0.1 90) (layer "B.SilkS")
       (effects (font (size 1 1) (thickness 0.15)) (justify mirror))
     )

Commit message: Update bring-up status: v0.2 USB-A host working
AnnePro2 FS HID keyboard fully enumerated on v0.2, key presses
confirmed 2026-08-12.

Also records PCB tweak: TP1 footprint drill 1.0mm→0.8mm with
alignment-library variant.

Co-Authored-By: Claude Sonnet 4.6 <noreply@anthropic.com>
Parts:
- TP1: footprint TestPoint:TestPoint_THTPad_D2.0mm_Drill1.0mm -> Alignment:TestPoint_THTPad_D2.0mm_Drill0.8mm_Align
Changed lines of the file:
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@@
     )
   )
-  (footprint "TestPoint:TestPoint_THTPad_D2.0mm_Drill1.0mm" (layer "F.Cu")
+  (footprint "Alignment:TestPoint_THTPad_D2.0mm_Drill0.8mm_Align" (layer "F.Cu")
     (at 112.2 52.1)
     (descr "THT pad as test Point, diameter 2.0mm, hole diameter 1.0mm")
@@
     (property "Sheetfile" "USB-pasthrough.kicad_sch")
     (property "Sheetname" "")
-    (attr exclude_from_pos_files)
-    (fp_text reference "TP1" (at -1.25 1.85) (layer "F.SilkS")
+    (attr exclude_from_pos_files exclude_from_bom)
+    (fp_text reference "TP1" (at 0 -1.998) (layer "F.SilkS")
       (effects (font (size 1 1) (thickness 0.15)))
     )
@@
     (fp_circle (center 0 0) (end 0 1.2) (layer "F.SilkS") (width 0.12) (fill none))
     (fp_circle (center 0 0) (end 1.5 0) (layer "F.CrtYd") (width 0.05) (fill none))
-    (pad "1" thru_hole circle (at 0 0) (size 2 2) (drill 1) (layers *.Cu *.Mask)
+    (pad "" smd circle (at 0 0) (size 0.8 0.8) (layers "F.Paste"))
+    (pad "1" thru_hole circle (at 0 0) (size 2 2) (drill 0.8) (layers *.Cu *.Mask)
       (net 2 "GND") (pinfunction "1") (pintype "passive"))
   )
